Commit message: follow_wall improved

File: urdf/new_robot2_laser.xacro (robot description, xacro)
@@ -161,6 +161,6 @@
 	      <origin xyz="0 0 0" rpy="0 0 0"/>
 	      <geometry>
-		     <box size="0.05 0.05 0.05"/>
-    <!-- <cylinder radius="0.05" length="0.05"/> -->
+		<!-- <box size="0.05 0.4 0.05"/> -->
+    <cylinder radius="0.05" length="0.05"/>
 	      </geometry>
 	    </collision>
@@ -168,6 +168,6 @@
 	      <origin xyz="0 0 0" rpy="0 0 0"/>
 	      <geometry>
-		     <box size="0.05 0.05 0.05"/>
-    <!-- <cylinder radius="0.05" length="0.05"/> -->
+		<!-- <box size="0.05 0.4 0.05"/> -->
+    <cylinder radius="0.05" length="0.05"/>
 	      </geometry>
 	      <material name="red">
@@ -183,5 +183,5 @@
   <joint name="hokuyo_joint" type="fixed">
 	    <axis xyz="0 1 0" />
-	    <origin xyz="0.25 0 0" rpy="0 0 0"/> <!-- 0 0.26 0-->
+	    <origin xyz="0.5 0 0" rpy="0 0 0"/> <!-- 0 0.26 0-->
 	    <parent link="link_chassis"/>
 	    <child link="hokuyo_link"/>
